File: IOB-I2C-PCA9685-PWM.sch (EAGLE design)
At the start: 12 parts, among them IC1 PCA9685PW, SW1 A0, SW2 A1

Commit message: normalized values
Parts:
- R1, R2, R3, R4, R5, R6: device SPCoast:R0805-RES -> SPCoast:R0603-RES
- SW1: value A0 -> SPSTx4
- SW2: value A1 -> SPSTx4
- U$1: value DOC-OSHW-LOGO-L -> OSHW
Changed lines of the file:
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@@
 <layer number="20" name="Dimension" color="15" fill="1" visible="no" active="no"/>
 <layer number="21" name="tPlace" color="19" fill="1" visible="no" active="no"/>
-<layer number="22" name="bPlace" color="22" fill="1" visible="no" active="no"/>
+<layer number="22" name="bPlace" color="17" fill="1" visible="no" active="no"/>
 <layer number="23" name="tOrigins" color="30" fill="1" visible="no" active="no"/>
 <layer number="24" name="bOrigins" color="15" fill="1" visible="no" active="no"/>
@@
 <layer number="46" name="Milling" color="35" fill="1" visible="no" active="no"/>
 <layer number="47" name="Measures" color="21" fill="1" visible="no" active="no"/>
-<layer number="48" name="Document" color="57" fill="1" visible="no" active="no"/>
+<layer number="48" name="Document" color="47" fill="1" visible="no" active="no"/>
 <layer number="49" name="Reference" color="48" fill="1" visible="no" active="no"/>
 <layer number="50" name="dxf" color="7" fill="1" visible="no" active="no"/>
-<layer number="51" name="tDocu" color="49" fill="1" visible="no" active="no"/>
+<layer number="51" name="tDocu" color="24" fill="1" visible="no" active="no"/>
 <layer number="52" name="bDocu" color="7" fill="1" visible="no" active="no"/>
 <layer number="53" name="tGND_GNDA" color="7" fill="9" visible="no" active="no"/>
@@
 <parts>
 <part name="FRAME1" library="MCP" deviceset="FRAME-LETTER" device=""/>
-<part name="U$1" library="SPCoast" deviceset="DOC-OSHW-LOGO-" device="L" value="DOC-OSHW-LOGO-L"/>
+<part name="U$1" library="SPCoast" deviceset="DOC-OSHW-LOGO-" device="L" value="OSHW"/>
 <part name="P+3" library="supply1" deviceset="VCC" device=""/>
 <part name="V9" library="supply2" deviceset="GND" device=""/>
-<part name="SW1" library="SPCoast" deviceset="SW_DIP-4" device="" value="A0"/>
-<part name="SW2" library="SPCoast" deviceset="SW_DIP-4" device="" value="A1"/>
+<part name="SW1" library="SPCoast" deviceset="SW_DIP-4" device="" value="SPSTx4"/>
+<part name="SW2" library="SPCoast" deviceset="SW_DIP-4" device="" value="SPSTx4"/>
 <part name="V5" library="supply2" deviceset="GND" device=""/>
 <part name="V6" library="supply2" deviceset="GND" device=""/>
@@
 <part name="V2" library="supply2" deviceset="GND" device=""/>
 <part name="V3" library="supply2" deviceset="GND" device=""/>
-<part name="R1" library="SPCoast" deviceset="R*" device="0805-RES" value="10k"/>
-<part name="R2" library="SPCoast" deviceset="R*" device="0805-RES" value="10k"/>
-<part name="R3" library="SPCoast" deviceset="R*" device="0805-RES" value="10k"/>
-<part name="R4" library="SPCoast" deviceset="R*" device="0805-RES" value="10k"/>
-<part name="R5" library="SPCoast" deviceset="R*" device="0805-RES" value="10k"/>
-<part name="R6" library="SPCoast" deviceset="R*" device="0805-RES" value="10k"/>
+<part name="R1" library="SPCoast" deviceset="R*" device="0603-RES" value="10k"/>
+<part name="R2" library="SPCoast" deviceset="R*" device="0603-RES" value="10k"/>
+<part name="R3" library="SPCoast" deviceset="R*" device="0603-RES" value="10k"/>
+<part name="R4" library="SPCoast" deviceset="R*" device="0603-RES" value="10k"/>
+<part name="R5" library="SPCoast" deviceset="R*" device="0603-RES" value="10k"/>
+<part name="R6" library="SPCoast" deviceset="R*" device="0603-RES" value="10k"/>
 <part name="P+4" library="supply1" deviceset="VCC" device=""/>
 </parts>
