File: IOB-I2C-PCA9685-PWM_array.brd (EAGLE design)
At the start: 108.7 x 112 mm, 39 parts, among them IC1X11 PCA9685PW, IC1X12 PCA9685PW, IC1X13 PCA9685PW, SW1X11 A0, SW1X12 A0, SW1X13 A0, SW2X11 A1, SW2X12 A1, SW2X13 A1

Commit message: added values for connectors
Parts:
- FID_LR, FID_UL: value (none) -> FIDUCIAL
- U$5X1: value (none) -> 10x10
Changed lines of the file:
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@@
 <element name="SW2X13" library="SPCoast" package="EDG-04" value="A1" x="46.355" y="74.93" rot="R180"/>
 <element name="U$1X13" library="SPCoast" package="OSHW-LOGO-L" value="DOC-OSHW-LOGO-L" x="76.835" y="75.057"/>
-<element name="U$5X1" library="SPCoast" package="BOARD-TEMPLATE-IOB-I2C-3X1-ARRAY" value="" x="0" y="0"/>
-<element name="FID_UL" library="SPCoast" package="FIDUCIAL_1MM" value="" x="5.08" y="91.44"/>
-<element name="FID_LR" library="SPCoast" package="FIDUCIAL_1MM" value="" x="93.98" y="8.89"/>
+<element name="U$5X1" library="SPCoast" package="BOARD-TEMPLATE-IOB-I2C-3X1-ARRAY" value="10x10" x="0" y="0"/>
+<element name="FID_UL" library="SPCoast" package="FIDUCIAL_1MM" value="FIDUCIAL" x="5.08" y="91.44"/>
+<element name="FID_LR" library="SPCoast" package="FIDUCIAL_1MM" value="FIDUCIAL" x="93.98" y="8.89"/>
 </elements>
 <signals>

Commit message: normalized values
Parts:
- SW1X11, SW1X12, SW1X13: value A0 -> SPSTx4
- SW2X11, SW2X12, SW2X13: value A1 -> SPSTx4
- U$1X11, U$1X12, U$1X13: value DOC-OSHW-LOGO-L -> OSHW
- U$5X1: value 10x10 -> BOARD
